Commit message: add palm pack collision

File: robots/hands/leap_hand/leap_hand_right.urdf (robot description, URDF)
Before this commit: robot leap_right, 22 links, 21 joints
Joints:
- removed joint 0
- removed joint 1
- removed joint 10
- removed joint 11
- removed joint 12
- removed joint 13
- removed joint 14
- removed joint 15
- removed joint 2
- removed joint 3
- removed joint 4
- removed joint 5
- removed joint 6
- removed joint 7
- removed joint 8
- removed joint 9
- added joint j00: type revolute, parent mcp_joint, child pip, origin xyz=-0.0122 0.03810 0.01450 rpy=-1.57079 0 1.57079, axis 0 0 -1, limit lower=-1.047 upper=1.047 effort=0.95 velocity=8.48
- added joint j01: type revolute, parent palm_lower, child mcp_joint, origin xyz=-0.0070 0.0230 -0.0187 rpy=1.57079 1.57079 0, axis 0 0 -1, limit lower=-0.314 upper=2.23 effort=0.95 velocity=8.48
- added joint j02: type revolute, parent pip, child dip, origin xyz=0.015 0.0143 -0.013 rpy=1.57079 -1.57079 0, axis 0 0 -1, limit lower=-0.506 upper=1.885 effort=0.95 velocity=8.48
- added joint j03: type revolute, parent dip, child fingertip, origin xyz=0 -0.0361 0.0002 rpy=0 0 0, axis 0 0 -1, limit lower=-0.366 upper=2.042 effort=0.95 velocity=8.48
- added joint j04: type revolute, parent mcp_joint_2, child pip_2, origin xyz=-0.0122 0.0381 0.0145 rpy=-1.57079 0 1.57079, axis 0 0 -1, limit lower=-1.047 upper=1.047 effort=0.95 velocity=8.48
- added joint j05: type revolute, parent palm_lower, child mcp_joint_2, origin xyz=-0.0071 -0.0224 -0.0187 rpy=1.57079 1.57079 0, axis 0 0 -1, limit lower=-0.314 upper=2.23 effort=0.95 velocity=8.48
- added joint j06: type revolute, parent pip_2, child dip_2, origin xyz=0.015 0.0143 -0.013 rpy=1.57079 -1.57079 0, axis 0 0 -1, limit lower=-0.506 upper=1.885 effort=0.95 velocity=8.48
- added joint j07: type revolute, parent dip_2, child fingertip_2, origin xyz=0 -0.0361 0.0002 rpy=0 0 0, axis 0 0 -1, limit lower=-0.366 upper=2.042 effort=0.95 velocity=8.48
- added joint j08: type revolute, parent mcp_joint_3, child pip_3, origin xyz=-0.0122 0.0381 0.0145 rpy=-1.57079 0 1.57079, axis 0 0 -1, limit lower=-1.047 upper=1.047 effort=0.95 velocity=8.48
- added joint j09: type revolute, parent palm_lower, child mcp_joint_3, origin xyz=-0.00709 -0.0678 -0.0187 rpy=1.57079 1.57079 0, axis 0 0 -1, limit lower=-0.314 upper=2.23 effort=0.95 velocity=8.48
- added joint j10: type revolute, parent pip_3, child dip_3, origin xyz=0.015 0.0143 -0.013 rpy=1.57079 -1.57079 0, axis 0 0 -1, limit lower=-0.506 upper=1.885 effort=0.95 velocity=8.48
- added joint j11: type revolute, parent dip_3, child fingertip_3, origin xyz=0 -0.03609 0.0002 rpy=0 0 0, axis 0 0 -1, limit lower=-0.366 upper=2.042 effort=0.95 velocity=8.48
- added joint j12: type revolute, parent palm_lower, child thumb_temp_base, origin xyz=-0.0693 -0.0012 -0.0216 rpy=0 1.57079 0, axis 0 0 -1, limit lower=-0.349 upper=2.094 effort=0.95 velocity=8.48
- added joint j13: type revolute, parent thumb_temp_base, child thumb_pip, origin xyz=0 0.0143 -0.013 rpy=1.57079 -1.57079 0, axis 0 0 -1, limit lower=-0.47 upper=2.443 effort=0.95 velocity=8.48
- added joint j14: type revolute, parent thumb_pip, child thumb_dip, origin xyz=0 0.0145 -0.017 rpy=-1.57079 0 0, axis 0 0 -1, limit lower=-1.20 upper=1.90 effort=0.95 velocity=8.48
- added joint j15: type revolute, parent thumb_dip, child thumb_fingertip, origin xyz=0 0.0466 0.0002 rpy=0 0 3.14159, axis 0 0 -1, limit lower=-1.34 upper=1.88 effort=0.95 velocity=8.48
